Commit message: last commit project

File: src/mob_rob_loca/urdf/edison.urdf (robot description, URDF)
Before this commit: robot Edison, 8 links, 7 joints
Joints:
- joint joint_marv: origin xyz=-0.11 0 0.075 rpy=0 0 0 -> xyz=-0.091 0 0.143 rpy=0 0 0; parent base_center -> base_link

Commit message: updates detection pc + rviz2 configuration (markers + cam urdf)

File: src/mob_rob_loca/urdf/edison.urdf (robot description, URDF)
Before this commit: robot Edison, 8 links, 7 joints
Links:
- added link camera, mass 0.1; collision box size=0.03 0.03 0.02; visual box size=0.03 0.03 0.02
Joints:
- added joint joint_cam: type fixed, parent base_link, child camera, origin xyz=0.1 0 0.143 rpy=0 0 0
